File: ai03-pcb-guide.sch (KiCad schematic (older format))
At the start: 24 parts, among them SW1 SW_Push, U1 ATmega32U4-AU, Y1 16MHz

Commit message: pcb-tut-1
Parts:
- MX1: value MX-NoLED -> MX1-NoLED
- MX2: renamed from MX3; value MX-NoLED -> MX2-NoLED
- MX3: renamed from MX2; value MX-NoLED -> MX3-NoLED
- MX4: value MX-NoLED -> MX4-NoLED
- renumbered D3 to D2, D2 to D3
Connections:
- net COL0: now also U1.29 (PB5)
- net COL1: now also U1.28 (PB4)
- net ROW0: now also U1.27 (PD7)
- net ROW1: now also U1.30 (PB6)
Changed lines of the file:
@@
 P 6850 2700
 F 0 "MX1" H 6883 2923 60  0000 C CNN
-F 1 "MX-NoLED" H 6883 2849 20  0000 C CNN
+F 1 "MX1-NoLED" H 6883 2849 20  0000 C CNN
 F 2 "MX_Alps_Hybrid:MX-1U-NoLED" H 6225 2675 60  0001 C CNN
 F 3 "" H 6225 2675 60  0001 C CNN
@@
 	6700 2850 6800 2850
 $Comp
-L MX_Alps_Hybrid:MX-NoLED MX3
+L MX_Alps_Hybrid:MX-NoLED MX2
 U 1 1 5D6C3814
 P 7500 2700
-F 0 "MX3" H 7533 2923 60  0000 C CNN
-F 1 "MX-NoLED" H 7533 2849 20  0000 C CNN
+F 0 "MX2" H 7533 2923 60  0000 C CNN
+F 1 "MX2-NoLED" H 7533 2849 20  0000 C CNN
 F 2 "MX_Alps_Hybrid:MX-1U-NoLED" H 6875 2675 60  0001 C CNN
 F 3 "" H 6875 2675 60  0001 C CNN
@@
 $EndComp
 $Comp
-L Device:D_Small D3
+L Device:D_Small D2
 U 1 1 5D6C381E
 P 7350 2950
-F 0 "D3" H 7350 3050 50  0000 R CNN
+F 0 "D2" H 7350 3050 50  0000 R CNN
 F 1 "SOD-123" H 7750 3050 50  0000 R CNN
 F 2 "Diode_SMD:D_SOD-123" V 7350 2950 50  0001 C CNN
@@
 	7350 2850 7450 2850
 $Comp
-L MX_Alps_Hybrid:MX-NoLED MX2
+L MX_Alps_Hybrid:MX-NoLED MX3
 U 1 1 5D6CD3C8
 P 6850 3350
-F 0 "MX2" H 6883 3573 60  0000 C CNN
-F 1 "MX-NoLED" H 6883 3499 20  0000 C CNN
+F 0 "MX3" H 6883 3573 60  0000 C CNN
+F 1 "MX3-NoLED" H 6883 3499 20  0000 C CNN
 F 2 "MX_Alps_Hybrid:MX-1U-NoLED" H 6225 3325 60  0001 C CNN
 F 3 "" H 6225 3325 60  0001 C CNN
@@
 $EndComp
 $Comp
-L Device:D_Small D2
+L Device:D_Small D3
 U 1 1 5D6CD3D2
 P 6700 3600
-F 0 "D2" H 6700 3700 50  0000 R CNN
+F 0 "D3" H 6700 3700 50  0000 R CNN
 F 1 "SOD-123" H 7100 3700 50  0000 R CNN
 F 2 "Diode_SMD:D_SOD-123" V 6700 3600 50  0001 C CNN
@@
 P 7500 3350
 F 0 "MX4" H 7533 3573 60  0000 C CNN
-F 1 "MX-NoLED" H 7533 3499 20  0000 C CNN
+F 1 "MX4-NoLED" H 7533 3499 20  0000 C CNN
 F 2 "MX_Alps_Hybrid:MX-1U-NoLED" H 6875 3325 60  0001 C CNN
 F 3 "" H 6875 3325 60  0001 C CNN
@@
 Text GLabel 7650 2200 1    50   Input ~ 0
 COL1
+Text GLabel 4150 1900 2    50   Input ~ 0
+COL1
+Text GLabel 4150 2000 2    50   Input ~ 0
+COL0
+Text GLabel 4150 3400 2    50   Input ~ 0
+ROW0
+Text GLabel 4150 2100 2    50   Input ~ 0
+ROW1
 $EndSCHEMATC
